File: Kicad/gpio-hc595-header/hc595-header.kicad_sch (KiCad schematic)
At the start: 7 parts, among them K1 GPIO IN, K2 GPIO OUT, K3 DATA OUTPUT, U1 74HC595-SOIC-16, U2 3M-SJ5376

Commit message: Update
Other:
- note added: "supprimer resistance reset"
Changed lines of the file:
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@@
     (effects (font (size 1.27 1.27)) (justify right bottom))
+  )
+  (text "supprimer resistance reset" (at 124.46 53.34 0)
+    (effects (font (size 2 2)) (justify left bottom))
   )
   (text "OUTPUT 2" (at 190.5 95.25 0)

Commit message: Update
Parts:
- removed R1: 10K, tronixio:RESISTOR-1206, symbol tronixio:R-1210
Connections:
- net VCC: now also U1.10 (~{MR})
Other:
- note removed: "supprimer resistance reset"
- moved on the sheet: K1, K2

Commit message: Update
Parts:
- removed C1: 100n, tronixio:CAPACITOR-1206, symbol tronixio:C-1206
- added C1: CAPACITOR-1206-100N, tronixio:CAPACITOR-1206, symbol tronixio:CAPACITOR-1206-100N
- K2: Name (none) -> SAMTEC-SSW-106-02-T-S-RA
- U2: footprint tronixio:zzz3M-SJ5376 -> tronixio:3M-SJ5376
Connections:
- net GND: now also C1.2
- net VCC: now also C1.1
Other:
- note removed: "*R6: 10K if NTC TH1 Not Populate."
- moved on the sheet: K1, K2, K3, U1

Commit message: Update
Parts:
- added C1: 10n, tronixio:CAPACITOR-SMD-1206, symbol tronixio:CAPACITOR-1206-10N
- added R1: 10K, tronixio:RESISTOR-SMD-1206, symbol tronixio:RESISTOR-1206-10K
- C2: renamed from C1; value CAPACITOR-1206-100N -> 100n; footprint tronixio:CAPACITOR-1206 -> tronixio:CAPACITOR-SMD-1206; Name 100n -> CAPACITOR-1206-100N
- K1: Name (none) -> HARWIN-254-M-1X06-RIGHT-ANGLE
- K3: value DATA OUTPUT -> DATA OUT; Name (none) -> HARWIN-254-M-1X08-VERTICAL
- U1: value 74HC595-SOIC-16 -> 74HC595; Name 74HC595 -> 74HC595-SOIC-16
Connections:
- net GND: now also C1.2
- net VCC renamed VDD
- net VDD: now also R1.1; no longer U1.10 (~{MR})
- new net: C1.1, R1.2, U1.10 (~{MR})
Other:
- note added: "VDD"
- note removed: "VCC"
- moved on the sheet: C2, K1, K2, K3, U1

Commit message: Update
Other:
- moved on the sheet: C2, K3, U1
