File: Kicad/gpio-hc595-header/hc595-header.kicad_sch (KiCad schematic)
At the start: 8 parts, among them K1 GPIO IN, K2 GPIO OUT, K3 DATA OUT, U1 74HC595, U2 3M-SJ5376

Commit message: Up
Parts:
- C1: symbol tronixio:CAPACITOR-1206-10N -> tronixio:CAPACITOR-1206-10N-50V-5P-X7R; Mouser 80-C1206C103M5R -> 80-C1206C103J5R; Tolerance 20% -> 5%
- C2: symbol tronixio:CAPACITOR-1206-100N -> tronixio:CAPACITOR-1206-100N-50V-5P-X7R; Mouser 80-C1206C104M5R -> 80-C1206C104J5R; Tolerance 20% -> 5%
- K2: symbol tronixio:SAMTEC-SSW-106-02-T-S-RA -> tronixio:SAMTEC-254-F-1X06-RIGHT-ANGLE; Mouser 200-SSW10602TSRA -> 200-SSW10603TSRA
- R1: symbol tronixio:RESISTOR-1206-10K -> tronixio:RESISTOR-1206-10K-5P
- U1: symbol tronixio:74HC595-SOIC-16 -> tronixio:NEXPERIA-74HC595-SOIC16; Mouser 771-AHC595D118 -> 771-AHC595D
Connections:
- net ~{OE}: now reaches K1.6, K2.1, U1.13 (~{OE})
- net STCP: now reaches K1.5, K2.2, U1.12 (STCP(CS))
- net SHCP: now reaches K1.4, K2.3, U1.11 (SHCP(SCK))
- net DS: now reaches K1.3, U1.14 (DS(DIN))
- net GND renamed POWER-GND
- net VDD renamed POWER-VBAT
Other:
- moved on the sheet: C1, C2, K1, K2, K3, R1, U1
