File: Kicad/gpio-hc595-header/hc595-header.kicad_pcb (KiCad board)
At the start: 2 copper layers, 50 x 25 mm, 13 parts, among them K1 GPIO IN, K2 GPIO OUT, K3 DATA OUTPUT, U1 74HC595-SOIC-16, U2 3M-SJ5376

Commit message: Update
Parts:
- removed R1: 10K, tronixio:RESISTOR-1206
Connections:
- U1 pad 10: Net-(R1-Pad1) -> VCC
Routing:
- net Net-(R1-Pad1): track 8.82 -> 0.00 mm
- net Q7S: track 19.0 -> 20.7 mm, vias 2 -> 1

Commit message: Updaet
Other:
- board text added: "+3V/5V"
- board text removed: "+3V-5V"
- board text removed: "TBOT Charger"
Changed lines of the file:
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@@
     (effects (font (size 1 1) (thickness 0.15)) (justify mirror))
   )
-  (gr_text "TBOT Charger" (at 132 68.5) (layer "B.SilkS")
+  (gr_text "GPIO 74HC595-HEADER" (at 132 68.5) (layer "B.SilkS")
     (effects (font (size 1 1) (thickness 0.2)) (justify mirror))
   )
@@
     (effects (font (size 1 1) (thickness 0.15)) (justify left))
   )
-  (gr_text "+3V-5V" (at 149.5 52.5) (layer "F.SilkS")
+  (gr_text "+3V/5V" (at 149.5 52.5) (layer "F.SilkS")
     (effects (font (size 1 1) (thickness 0.15)) (justify right))
   )

Commit message: Update
Routing:
- net Net-(K1-Pad6): track 37.7 -> 39.7 mm
- net Net-(K1-Pad5): track 39.9 -> 40.8 mm
Other:
- outline, holes or cut-outs redrawn
Changed lines of the file:
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@@
       (layer "F.SilkS" (type "Top Silk Screen") (color "White"))
       (layer "F.Paste" (type "Top Solder Paste"))
-      (layer "F.Mask" (type "Top Solder Mask") (color "Purple") (thickness 0.01))
+      (layer "F.Mask" (type "Top Solder Mask") (color "Black") (thickness 0.01))
       (layer "F.Cu" (type "copper") (thickness 0.035))
       (layer "dielectric 1" (type "prepreg") (thickness 1.51) (material "FR4") (epsilon_r 4.5) (loss_tangent 0.02))
       (layer "B.Cu" (type "copper") (thickness 0.035))
-      (layer "B.Mask" (type "Bottom Solder Mask") (color "Purple") (thickness 0.01))
+      (layer "B.Mask" (type "Bottom Solder Mask") (color "Black") (thickness 0.01))
       (layer "B.Paste" (type "Bottom Solder Paste"))
       (layer "B.SilkS" (type "Bottom Silk Screen") (color "White"))
@@
     )
   )
-  (gr_rect (start 101 54) (end 105 52) (layer "F.Cu") (width 0.1) (fill none))
-  (gr_line (start 103 54) (end 103 52) (layer "F.Cu") (width 0.1))
-  (gr_line (start 103 54) (end 103 52) (layer "B.Cu") (width 0.1))
-  (gr_rect (start 101 54) (end 105 52) (layer "B.Cu") (width 0.1) (fill none))
+  (gr_rect (start 102 54) (end 106 52) (layer "F.Cu") (width 0.1) (fill none))
+  (gr_line (start 104 54) (end 104 52) (layer "F.Cu") (width 0.1))
+  (gr_line (start 104 54) (end 104 52) (layer "B.Cu") (width 0.1))
+  (gr_rect (start 102 54) (end 106 52) (layer "B.Cu") (width 0.1) (fill none))
   (gr_circle (center 133.5 66) (end 133.75 66) (layer "F.SilkS") (width 0.1) (fill solid))
   (gr_line (start 90 53.5) (end 90 48.5) (layer "Dwgs.User") (width 0.05))
@@
   (gr_line (start 160 76) (end 159.5 76) (layer "Dwgs.User") (width 0.05))
   (gr_circle (center 90 51) (end 91 51) (layer "Dwgs.User") (width 0.05) (fill none))
-  (gr_arc (start 100 52) (mid 100.292893 51.292893) (end 101 51) (layer "Edge.Cuts") (width 0.15))
-  (gr_line (start 150 51) (end 101 51) (layer "Edge.Cuts") (width 0.15))
-  (gr_line (start 100 52) (end 100 75) (layer "Edge.Cuts") (width 0.15))
-  (gr_line (start 101 76) (end 150 76) (layer "Edge.Cuts") (width 0.15))
+  (gr_line (start 150 51) (end 102 51) (layer "Edge.Cuts") (width 0.15))
+  (gr_line (start 100 53) (end 100 74) (layer "Edge.Cuts") (width 0.15))
+  (gr_line (start 102 76) (end 150 76) (layer "Edge.Cuts") (width 0.15))
+  (gr_arc (start 100 53) (mid 100.585786 51.585786) (end 102 51) (layer "Edge.Cuts") (width 0.15))
+  (gr_arc (start 102 76) (mid 100.585786 75.414214) (end 100 74) (layer "Edge.Cuts") (width 0.15))
   (gr_line (start 150 76) (end 150 51) (layer "Edge.Cuts") (width 0.15))
-  (gr_arc (start 101 76) (mid 100.292893 75.707107) (end 100 75) (layer "Edge.Cuts") (width 0.15))
-  (gr_text "1" (at 102 53) (layer "F.Cu")
+  (gr_text "1" (at 103 53) (layer "F.Cu")
     (effects (font (size 1 1) (thickness 0.15)))
   )
-  (gr_text "2" (at 104 53) (layer "B.Cu")
+  (gr_text "2" (at 105 53) (layer "B.Cu")
     (effects (font (size 1 1) (thickness 0.15)) (justify mirror))
   )
@@
     (effects (font (size 1 1) (thickness 0.15)))
   )
-  (gr_text "202201 - Rev.A" (at 100.5 74.5) (layer "F.SilkS")
+  (gr_text "202201 - Rev.A" (at 101.25 74.5) (layer "F.SilkS")
     (effects (font (size 1 1) (thickness 0.15)) (justify left))
   )
@@
     (effects (font (size 1 1) (thickness 0.15)))
   )
-  (gr_text "GPIO 74HC595-HEADER" (at 100.5 72.5) (layer "F.SilkS")
+  (gr_text "GPIO 74HC595-HEADER" (at 101.25 72.5) (layer "F.SilkS")
     (effects (font (size 1 1) (thickness 0.2)) (justify left))
   )
@@
   (via (at 117 62.23) (size 0.6) (drill 0.3) (layers "F.Cu" "B.Cu") (net 3))
   (segment (start 117 62.23) (end 110 62.23) (width 0.5) (layer "B.Cu") (net 3))
-  (segment (start 134.5 67) (end 133 68.5) (width 0.5) (layer "F.Cu") (net 4))
+  (segment (start 129.905 70.095) (end 129.905 71.75) (width 0.5) (layer "F.Cu") (net 4))
+  (segment (start 134.5 66.5) (end 132.5 68.5) (width 0.5) (layer "F.Cu") (net 4))
+  (segment (start 132.5 68.5) (end 131.5 68.5) (width 0.5) (layer "F.Cu") (net 4))
   (segment (start 131.5 68.5) (end 129.905 70.095) (width 0.5) (layer "F.Cu") (net 4))
-  (segment (start 129.905 70.095) (end 129.905 71.75) (width 0.5) (layer "F.Cu") (net 4))
-  (segment (start 133 68.5) (end 131.5 68.5) (width 0.5) (layer "F.Cu") (net 4))
-  (via (at 134.5 67) (size 0.6) (drill 0.3) (layers "F.Cu" "B.Cu") (net 4))
-  (segment (start 134.5 67) (end 141.003 67) (width 0.5) (layer "B.Cu") (net 4))
-  (segment (start 141.003 67) (end 145.773 62.23) (width 0.5) (layer "B.Cu") (net 4))
+  (via (at 134.5 66.5) (size 0.6) (drill 0.3) (layers "F.Cu" "B.Cu") (net 4))
+  (segment (start 141.503 66.5) (end 145.773 62.23) (width 0.5) (layer "B.Cu") (net 4))
+  (segment (start 134.5 66.5) (end 141.503 66.5) (width 0.5) (layer "B.Cu") (net 4))
   (segment (start 126.095 71.75) (end 126.095 68) (width 0.5) (layer "F.Cu") (net 5))
   (via (at 126.095 68) (size 0.6) (drill 0.3) (layers "F.Cu" "B.Cu") (net 5))
@@
   (segment (start 127.365 71.75) (end 127.365 69) (width 0.5) (layer "F.Cu") (net 6))
   (via (at 127.365 69) (size 0.6) (drill 0.3) (layers "F.Cu" "B.Cu") (net 6))
-  (segment (start 145.773 67.31) (end 144.083 69) (width 0.5) (layer "B.Cu") (net 6))
-  (segment (start 144.083 69) (end 111.69 69) (width 0.5) (layer "B.Cu") (net 6))
-  (segment (start 111.69 69) (end 110 67.31) (width 0.5) (layer "B.Cu") (net 6))
+  (segment (start 110 67.31) (end 112.19 69.5) (width 0.5) (layer "B.Cu") (net 6))
+  (segment (start 129.5 69) (end 130 69.5) (width 0.5) (layer "B.Cu") (net 6))
+  (segment (start 112.19 69.5) (end 126.865 69.5) (width 0.5) (layer "B.Cu") (net 6))
+  (segment (start 143.583 69.5) (end 145.773 67.31) (width 0.5) (layer "B.Cu") (net 6))
+  (segment (start 127.365 69) (end 129.5 69) (width 0.5) (layer "B.Cu") (net 6))
+  (segment (start 126.865 69.5) (end 127.365 69) (width 0.5) (layer "B.Cu") (net 6))
+  (segment (start 130 69.5) (end 143.583 69.5) (width 0.5) (layer "B.Cu") (net 6))
   (segment (start 128.635 71.75) (end 128.635 69.85) (width 0.5) (layer "F.Cu") (net 7))
   (via (at 128.635 69.85) (size 0.6) (drill 0.3) (layers "F.Cu" "B.Cu") (net 7))
-  (segment (start 145.773 69.85) (end 110 69.85) (width 0.5) (layer "B.Cu") (net 7))
+  (segment (start 144.623 71) (end 129.5 71) (width 0.5) (layer "B.Cu") (net 7))
+  (segment (start 127.485 71) (end 128.4925 69.9925) (width 0.5) (layer "B.Cu") (net 7))
+  (segment (start 110 69.85) (end 111.15 71) (width 0.5) (layer "B.Cu") (net 7))
+  (segment (start 129.5 71) (end 128.4925 69.9925) (width 0.5) (layer "B.Cu") (net 7))
+  (segment (start 128.4925 69.9925) (end 128.635 69.85) (width 0.5) (layer "B.Cu") (net 7))
+  (segment (start 111.15 71) (end 127.485 71) (width 0.5) (layer "B.Cu") (net 7))
+  (segment (start 145.773 69.85) (end 144.623 71) (width 0.5) (layer "B.Cu") (net 7))
   (segment (start 119.11 57.61) (end 124.825 63.325) (width 0.5) (layer "F.Cu") (net 8))
   (segment (start 124.825 63.325) (end 124.825 66.25) (width 0.5) (layer "F.Cu") (net 8))

Commit message: Update
Parts:
- removed kibuzzard-62B2FDD2: G***, kibuzzard-62B2FDD2
- removed kibuzzard-62B2FE3C: G***, kibuzzard-62B2FE3C
- added C2: 100n, tronixio:CAPACITOR-SMD-1206, F.Cu at (121.5, 69.0)
- added R1: 10K, tronixio:RESISTOR-SMD-1206, F.Cu at (119.0, 69.0)
- added kibuzzard-62EAC0B7: G***, kibuzzard-62EAC0B7, F.Cu at (142.2, 57.1)
- added kibuzzard-62EAC0C0: G***, kibuzzard-62EAC0C0, F.Cu at (113.5, 57.1)
- C1: value 100n -> 10n; footprint tronixio:CAPACITOR-1206 -> tronixio:CAPACITOR-SMD-1206
- K3: value DATA OUTPUT -> DATA OUT
- U1: value 74HC595-SOIC-16 -> 74HC595
- U2: footprint tronixio:zzz3M-SJ5376 -> tronixio:3M-SJ5376
- moved C1 5.00 mm to (116.5, 69.0), turned to -90 degrees
Connections:
- C1 pad 1: VCC -> Net-(C1-Pad1)
- K1 pad 1: VCC -> VDD
- K2 pad 6: VCC -> VDD
- U1 pad 10: VCC -> Net-(C1-Pad1)
- U1 pad 16: VCC -> VDD
Routing:
- net VDD: track 0.00 -> 76.0 mm, vias 0 -> 2
- net VCC: track 72.5 -> 0.00 mm
- net Net-(C1-Pad1): track 0.00 -> 11.5 mm
- net Q7S: track 20.7 -> 22.4 mm, vias 1 -> 0
- net GND: track 4.63 -> 6.13 mm, vias 1 -> 2
Other:
- board text added: "GPIO - 74HC595-HEADER - Rev.A - (01/2022) - Scale 100%"
- board text added: "~{OE}"
- board text removed: "GPIO 74HC595-HEADER - Rev.A - (01/2022) - Scale 100%"
- board text removed: "OE"

Commit message: Update
Other:
- board text added: "+3V/+5V"
- board text added: "70mA"
- board text removed: "+3V/5V"
- board text removed: "5mA"
Changed lines of the file:
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@@
     (effects (font (size 1 1) (thickness 0.15)) (justify left))
   )
-  (gr_text "+3V/5V" (at 149.5 52.5) (layer "F.SilkS")
+  (gr_text "+3V/+5V" (at 149.5 52.5) (layer "F.SilkS")
     (effects (font (size 1 1) (thickness 0.15)) (justify right))
   )
@@
     (effects (font (size 1 1) (thickness 0.15)) (justify left))
   )
-  (gr_text "5mA" (at 149.5 54.5) (layer "F.SilkS")
+  (gr_text "70mA" (at 149.5 54.5) (layer "F.SilkS")
     (effects (font (size 1 1) (thickness 0.15)) (justify right))
   )
