File: Kicad/gpio-hc595-header/hc595-header.kicad_pcb (KiCad board)
At the start: 2 copper layers, 50 x 25 mm, 14 parts, among them K1 GPIO IN, K2 GPIO OUT, K3 DATA OUT, U1 74HC595, U2 3M-SJ5376

Commit message: Up
Connections:
- net GND renamed POWER-GND
- net Net-(K1-Pad3) renamed DS
- net Net-(K1-Pad4) renamed SHCP
- net Net-(K1-Pad5) renamed STCP
- net Net-(K1-Pad6) renamed ~{OE}
- net VDD renamed POWER-VBAT
