File: Kicad/gpio-hc595-led/hc595-led.kicad_pcb (KiCad board)
At the start: 2 copper layers, 50 x 25 mm, 24 parts, among them K1 GPIO IN, K2 GPIO OUT, U1 74HC595-SOIC-16, U2 3M-SJ5376

Commit message: Update
Parts:
- removed R1: 10K, tronixio:RESISTOR-1206
Connections:
- U1 pad 10: Net-(R1-Pad1) -> VCC
Routing:
- net Net-(R1-Pad1): track 8.82 -> 0.00 mm
- net Q7S: track 19.0 -> 18.5 mm, vias 2 -> 1

Commit message: Updaet
Other:
- board text added: "+3V/5V"
- board text removed: "+3V-5V"
- board text removed: "TBOT Charger"
Changed lines of the file:
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@@
     (effects (font (size 1 1) (thickness 0.15)) (justify mirror))
   )
-  (gr_text "TBOT Charger" (at 132 68) (layer "B.SilkS")
+  (gr_text "GPIO 74HC595-LED" (at 132 68) (layer "B.SilkS")
     (effects (font (size 1 1) (thickness 0.2)) (justify mirror))
   )
@@
     (effects (font (size 1 1) (thickness 0.15)) (justify left))
   )
-  (gr_text "+3V-5V" (at 149.5 52.5) (layer "F.SilkS")
+  (gr_text "+3V/5V" (at 149.5 52.5) (layer "F.SilkS")
     (effects (font (size 1 1) (thickness 0.15)) (justify right))
   )

Commit message: Update
Parts:
- added kibuzzard-62B79DF9: G***, kibuzzard-62B79DF9, F.Cu at (112.8, 57.1)
- added kibuzzard-62B79E59: G***, kibuzzard-62B79E59, F.Cu at (112.8, 59.7)
- added kibuzzard-62B79EB2: G***, kibuzzard-62B79EB2, F.Cu at (143.0, 57.1)
- added kibuzzard-62B79EC3: G***, kibuzzard-62B79EC3, F.Cu at (143.0, 59.7)

Commit message: Update
Routing:
- net Net-(K1-Pad6): track 37.7 -> 39.6 mm
- net Net-(K1-Pad5): track 39.9 -> 40.8 mm
Other:
- outline, holes or cut-outs redrawn

Commit message: Update
Changed lines of the file:
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@@
       (layer "F.SilkS" (type "Top Silk Screen") (color "White"))
       (layer "F.Paste" (type "Top Solder Paste"))
-      (layer "F.Mask" (type "Top Solder Mask") (color "Purple") (thickness 0.01))
+      (layer "F.Mask" (type "Top Solder Mask") (color "Black") (thickness 0.01))
       (layer "F.Cu" (type "copper") (thickness 0.035))
       (layer "dielectric 1" (type "prepreg") (thickness 1.51) (material "FR4") (epsilon_r 4.5) (loss_tangent 0.02))
       (layer "B.Cu" (type "copper") (thickness 0.035))
-      (layer "B.Mask" (type "Bottom Solder Mask") (color "Purple") (thickness 0.01))
+      (layer "B.Mask" (type "Bottom Solder Mask") (color "Black") (thickness 0.01))
       (layer "B.Paste" (type "Bottom Solder Paste"))
       (layer "B.SilkS" (type "Bottom Silk Screen") (color "White"))
@@
     (effects (font (size 0.8 0.8) (thickness 0.1)))
   )
-  (gr_text "202201 - Rev.A" (at 100.5 74.5) (layer "F.SilkS")
+  (gr_text "202201 - Rev.A" (at 101.5 74.5) (layer "F.SilkS")
     (effects (font (size 1 1) (thickness 0.15)) (justify left))
   )
@@
     (effects (font (size 1 1) (thickness 0.15)) (justify right))
   )
-  (gr_text "GPIO 74HC595-LED" (at 100.5 72.5) (layer "F.SilkS")
+  (gr_text "GPIO 74HC595-LED" (at 101.5 72.5) (layer "F.SilkS")
     (effects (font (size 1 1) (thickness 0.2)) (justify left))
   )

Commit message: Update
Parts:
- added C1: 10n, tronixio:CAPACITOR-SMD-1206, F.Cu at (116.5, 69.0)
- added R1: 10K, tronixio:RESISTOR-SMD-1206, F.Cu at (119.0, 69.0)
- C2: renamed from C1; footprint tronixio:CAPACITOR-1206 -> tronixio:CAPACITOR-SMD-1206
- LED1, LED2, LED3, LED4, LED5, LED6, LED7, LED8: footprint tronixio:LED-1206 -> tronixio:LED-SMD-1206
- R2, R3, R4, R5, R6, R7, R8, R9: footprint tronixio:RESISTOR-1206 -> tronixio:RESISTOR-SMD-1206
- U1: value 74HC595-SOIC-16 -> 74HC595
- U2: footprint tronixio:zzz3M-SJ5376 -> tronixio:3M-SJ5376
Connections:
- C2 pad 1: VCC -> VDD
- K1 pad 1: VCC -> VDD
- K2 pad 6: VCC -> VDD
- U1 pad 10: VCC -> Net-(C1-Pad1)
- U1 pad 16: VCC -> VDD
Routing:
- net VDD: track 0.00 -> 74.9 mm, vias 0 -> 2
- net VCC: track 71.4 -> 0.00 mm
- net Net-(C1-Pad1): track 0.00 -> 11.5 mm
- net Q7S: track 18.5 -> 22.7 mm, vias 1 -> 0
- net GND: track 32.6 -> 34.3 mm, vias 3 -> 4
Other:
- board text added: "GPIO - 74HC595-LED - Rev.A - (01/2022) - Scale 100%"
- board text added: "~{OE}"
- board text removed: "GPIO 74HC595-LED - Rev.A - (01/2022) - Scale 100%"
- board text removed: "OE"

Commit message: Update
Parts:
- moved C1 29.1 mm to (142.5, 82.0)
- moved C2 29.1 mm to (147.5, 82.0)
- moved G*** 29.1 mm to (174.0, 86.5)
- moved GT 29.1 mm to (158.0, 70.5)
- moved K1 29.1 mm to (171.8, 70.2)
- moved K2 29.1 mm to (136.0, 82.8)
- moved LED1 29.1 mm to (166.2, 67.5)
- moved LED2 29.1 mm to (162.8, 67.5)
- moved LED3 29.1 mm to (159.2, 67.5)
- moved LED4 29.1 mm to (155.8, 67.5)
- moved LED5 29.1 mm to (152.2, 67.5)
- moved LED6 29.1 mm to (148.8, 67.5)
- moved LED7 29.1 mm to (145.2, 67.5)
- moved LED8 29.1 mm to (141.8, 67.5)
- moved R1 29.1 mm to (145.0, 82.0)
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Other:
- board text added: "+3V/+5V"
- board text added: "70mA"
- board text removed: "+3V/5V"
- board text removed: "20mA"
