File: Kicad/gpio-breadbaord/main.kicad_pcb (KiCad board)
At the start: 2 copper layers, 98 x 60 mm, 12 parts, among them K1 GPIO IN, K2 GPIO OUT #1, K3 GPIO OUT #2, K4 GPIO #1, K5 GPIO #2

Commit message: Up
Parts:
- removed the GT at (149.0, 67.5)
- K1, K2, K3: footprint tronixio:HARWIN-M20-999154x -> tronixio:HARWIN-M20-999164x
- moved K2 0.78 mm to (103.5, 55.9)
- moved K3 0.78 mm to (194.5, 55.9)
- moved H2 0.50 mm to (195.5, 102.0)
Routing:
- net Net-(K1-Pad16): track 0.00 -> 138.0 mm, vias 0 -> 1
- net Net-(K1-Pad1): track 123.1 -> 121.6 mm
- net Net-(K1-Pad2): track 128.2 -> 126.7 mm
- net Net-(K1-Pad14): track 133.7 -> 133.0 mm
- net Net-(K1-Pad9): track 121.0 -> 120.3 mm
- net Net-(K1-Pad8): track 118.5 -> 117.7 mm
- net Net-(K1-Pad6): track 113.4 -> 112.6 mm
- net Net-(K1-Pad5): track 110.9 -> 110.1 mm
- net Net-(K1-Pad4): track 108.3 -> 107.6 mm
- net Net-(K1-Pad15): track 136.3 -> 135.5 mm
- net Net-(K1-Pad12): track 128.7 -> 127.9 mm
- net Net-(K1-Pad11): track 126.1 -> 125.3 mm
- net Net-(K1-Pad10): track 123.6 -> 122.8 mm
- net Net-(K1-Pad7): track 116.0 -> 115.2 mm
- net Net-(K1-Pad3): track 105.8 -> 105.0 mm
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