File: Kicad/gpio-breadbaord/main.kicad_pcb (KiCad board)
At the start: 2 copper layers, 98 x 60 mm, 11 parts, among them K1 GPIO IN, K2 GPIO OUT #1, K3 GPIO OUT #2, K4 GPIO #1, K5 GPIO #2

Commit message: Update Kicad 8
Parts:
- H1, H2, H3, H4: footprint tronixio:MOUNTING-HOLE-2.5MM-MASK -> tronixio:MOUNTING-HOLE-3MM-MASK
Other:
- outline, holes or cut-outs redrawn
- board text added: "GPIO - MODULE-BREADBOARD 400 - Rev.A - (01/2023) - Scale 100%"
- board text added: "GPIO MODULE BREADBOARD 400"
- board text removed: "GPIO - MODULE-BREADBOARD - Rev.A - (01/2023) - Scale 100%"
- board text removed: "GPIO MODULE BREADBOARD"

Commit message: Update Breadboard
Other:
- board text added: "012023 - Rev.A"
- board text removed: "202301 - Rev.A"

Commit message: Up
Parts:
- K2: value GPIO OUT #1 -> GPIO OUT #3
- K3: value GPIO OUT #2 -> GPIO OUT #1; footprint tronixio:HARWIN-M20-999164x -> tronixio:HARWIN-M20-999064x
- K4: value GPIO #1 -> GPIO OUT #4; footprint tronixio:HARWIN-M20-999064x -> tronixio:HARWIN-M20-999164x
- K5: value GPIO #2 -> GPIO OUT #2
- moved K3 40.5 mm to (155.0, 47.0), turned to 90 degrees
- moved K4 40.5 mm to (194.5, 55.9), turned to 0 degrees
Connections:
- K3 pad 2: Net-(K1-Pin_2) -> Net-(K1-Pin_1)
- K3 pad 3: Net-(K1-Pin_3) -> Net-(K1-Pin_1)
- K3 pad 4: Net-(K1-Pin_4) -> Net-(K1-Pin_1)
- K3 pad 5: Net-(K1-Pin_5) -> Net-(K1-Pin_1)
- K3 pad 6: Net-(K1-Pin_6) -> Net-(K1-Pin_1)
- K4 pad 2: Net-(K1-Pin_1) -> Net-(K1-Pin_2)
- K4 pad 3: Net-(K1-Pin_1) -> Net-(K1-Pin_3)
- K4 pad 4: Net-(K1-Pin_1) -> Net-(K1-Pin_4)
- K4 pad 5: Net-(K1-Pin_1) -> Net-(K1-Pin_5)
- K4 pad 6: Net-(K1-Pin_1) -> Net-(K1-Pin_6)
Other:
- board text added: "2024Q4 - Rev.A"
- board text added: "GPIO - BREADBOARD 400 - Rev.A - (Q4/2024) - Scale 100%"
- board text added: "GPIO BREADBOARD 400"
- board text removed: "012023 - Rev.A"
- board text removed: "GPIO - MODULE-BREADBOARD 400 - Rev.A - (01/2023) - Scale 100%"
- board text removed: "GPIO MODULE BREADBOARD 400"

Commit message: Up
Parts:
- K4: footprint tronixio:HARWIN-M20-999164x -> tronixio:HARWIN-M20-782164x
