File: Kicad/gpio-breadbaord/main.kicad_sch (KiCad schematic)
At the start: 10 parts, among them K1 GPIO IN, K2 GPIO OUT #1, K3 GPIO OUT #2, K4 GPIO #1, K5 GPIO #2

Commit message: Up
Parts:
- K1, K2, K3: footprint tronixio:HARWIN-M20-999154x -> tronixio:HARWIN-M20-999164x; symbol tronixio:HARWIN-254-M-1X15-VERTICAL -> tronixio:HARWIN-254-M-1X16-VERTICAL; Mouser 855-M20-999154 -> 855-M20-999164; Name HARWIN-254-M-1X15-VERTICAL -> HARWIN-254-M-1X16-VERTICAL
Connections:
- new net: K1.16 (Pin_16), K2.16 (Pin_16), K3.16 (Pin_16)
Other:
- note added: "1"
- note added: "10"
- note added: "11"
- note added: "12"
- note added: "13"
- note added: "14"
- note added: "15"
- note added: "2"
- note added: "3"
- note added: "4"
- note added: "5"
- note added: "6"
- note added: "7"
- note added: "8"
- note added: "9"
- note removed: "DS"
- note removed: "GND"
- note removed: "SHCP"
- note removed: "STCP"
- note removed: "VDD"
- note removed: "~{OE}"
Changed lines of the file:
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@@
   (junction (at 180.34 83.82) (diameter 0) (color 0 0 0 0)
   )
+  (junction (at 152.4 71.12) (diameter 0) (color 0 0 0 0)
+  )
   (junction (at 121.92 40.64) (diameter 0) (color 0 0 0 0)
   )
@@
     (stroke (width 0) (type default) (color 0 0 0 0))
   )
+  (wire (pts (xy 152.4 116.84) (xy 152.4 71.12))
+    (stroke (width 0) (type default) (color 0 0 0 0))
+  )
   (wire (pts (xy 124.46 88.9) (xy 124.46 43.18))
     (stroke (width 0) (type default) (color 0 0 0 0))
@@
     (stroke (width 0) (type default) (color 0 0 0 0))
   )
+  (wire (pts (xy 111.76 116.84) (xy 152.4 116.84))
+    (stroke (width 0) (type default) (color 0 0 0 0))
+  )
   (wire (pts (xy 111.76 93.98) (xy 129.54 93.98))
     (stroke (width 0) (type default) (color 0 0 0 0))
@@
     (stroke (width 0) (type default) (color 0 0 0 0))
   )
+  (wire (pts (xy 152.4 71.12) (xy 111.76 71.12))
+    (stroke (width 0) (type default) (color 0 0 0 0))
+  )
   (wire (pts (xy 149.86 68.58) (xy 187.96 68.58))
     (stroke (width 0) (type default) (color 0 0 0 0))
   )
+  (wire (pts (xy 152.4 71.12) (xy 187.96 71.12))
+    (stroke (width 0) (type default) (color 0 0 0 0))
+  )
   (wire (pts (xy 111.76 104.14) (xy 139.7 104.14))
     (stroke (width 0) (type default) (color 0 0 0 0))
@@
     (stroke (width 0) (type default) (color 0 0 0 0))
   )
-  (text "SHCP" (at 106.68 41.91 180)
-    (effects (font (size 1.27 1.27)) (justify right bottom))
-  )
-  (text "~{OE}" (at 106.68 46.99 180)
-    (effects (font (size 1.27 1.27)) (justify right bottom))
-  )
-  (text "VDD" (at 106.68 34.29 180)
-    (effects (font (size 1.27 1.27)) (justify right bottom))
-  )
-  (text "DS" (at 106.68 39.37 180)
-    (effects (font (size 1.27 1.27)) (justify right bottom))
-  )
-  (text "STCP" (at 106.68 44.45 180)
-    (effects (font (size 1.27 1.27)) (justify right bottom))
-  )
-  (text "GND" (at 106.68 36.83 180)
-    (effects (font (size 1.27 1.27)) (justify right bottom))
-  )
-  (symbol (lib_id "tronixio:HARWIN-254-M-1X15-VERTICAL") (at 190.5 33.02 0) (unit 1)
+  (text "4" (at 106.68 41.91 180)
+    (effects (font (size 1.27 1.27)) (justify right bottom))
+  )
+  (text "11" (at 106.68 59.69 180)
+    (effects (font (size 1.27 1.27)) (justify right bottom))
+  )
+  (text "10" (at 106.68 57.15 180)
+    (effects (font (size 1.27 1.27)) (justify right bottom))
+  )
+  (text "12" (at 106.68 62.23 180)
+    (effects (font (size 1.27 1.27)) (justify right bottom))
+  )
+  (text "9" (at 106.68 54.61 180)
+    (effects (font (size 1.27 1.27)) (justify right bottom))
+  )
+  (text "6" (at 106.68 46.99 180)
+    (effects (font (size 1.27 1.27)) (justify right bottom))
+  )
+  (text "1" (at 106.68 34.29 180)
+    (effects (font (size 1.27 1.27)) (justify right bottom))
+  )
+  (text "3" (at 106.68 39.37 180)
+    (effects (font (size 1.27 1.27)) (justify right bottom))
+  )
+  (text "15" (at 106.68 69.85 180)
+    (effects (font (size 1.27 1.27)) (justify right bottom))
+  )
+  (text "7" (at 106.68 49.53 180)
+    (effects (font (size 1.27 1.27)) (justify right bottom))
+  )
+  (text "5" (at 106.68 44.45 180)
+    (effects (font (size 1.27 1.27)) (justify right bottom))
+  )
+  (text "13" (at 106.68 64.77 180)
+    (effects (font (size 1.27 1.27)) (justify right bottom))
+  )
+  (text "2" (at 106.68 36.83 180)
+    (effects (font (size 1.27 1.27)) (justify right bottom))
+  )
+  (text "8" (at 106.68 52.07 180)
+    (effects (font (size 1.27 1.27)) (justify right bottom))
+  )
+  (text "14" (at 106.68 67.31 180)
+    (effects (font (size 1.27 1.27)) (justify right bottom))
+  )
+  (symbol (lib_id "tronixio:HARWIN-254-M-1X16-VERTICAL") (at 190.5 33.02 0) (unit 1)
     (in_bom yes) (on_board yes)
     (property "Reference" "K2" (id 0) (at 190.5 30.48 0)
       (effects (font (size 1.15 1.15)))
     )
-    (property "Value" "GPIO OUT #1" (id 1) (at 190.5 71.12 0)
-      (effects (font (size 1.15 1.15)))
-    )
-    (property "Footprint" "tronixio:HARWIN-M20-999154x" (id 2) (at 190.5 76.2 0)
-      (effects (font (size 1 1)) hide)
-    )
-    (property "Datasheet" "https://www.harwin.com/products/M20-9991546/" (id 3) (at 190.5 78.74 0)
-      (effects (font (size 1 1)) hide)
-    )
-    (property "Mouser" "855-M20-999154" (id 4) (at 190.5 81.28 0)
-      (effects (font (size 1 1)) hide)
-    )
-    (property "Name" "HARWIN-254-M-1X15-VERTICAL" (id 5) (at 190.5 73.66 0)
+    (property "Value" "GPIO OUT #1" (id 1) (at 190.5 73.66 0)
+      (effects (font (size 1.15 1.15)))
+    )
+    (property "Footprint" "tronixio:HARWIN-M20-999164x" (id 2) (at 190.5 78.74 0)
+      (effects (font (size 1 1)) hide)
+    )
+    (property "Datasheet" "https://www.harwin.com/products/M20-9991646/" (id 3) (at 190.5 81.28 0)
+      (effects (font (size 1 1)) hide)
+    )
+    (property "Mouser" "855-M20-999164" (id 4) (at 190.5 83.82 0)
+      (effects (font (size 1 1)) hide)
+    )
+    (property "Name" "HARWIN-254-M-1X16-VERTICAL" (id 5) (at 190.5 76.2 0)
       (effects (font (size 1 1)) hide)
     )
@@
     (pin "14")
     (pin "15")
+    (pin "16")
     (pin "2")
     (pin "3")
@@
     )
   )
-  (symbol (lib_id "tronixio:HARWIN-254-M-1X15-VERTICAL") (at 109.22 33.02 0) (mirror y) (unit 1)
+  (symbol (lib_id "tronixio:HARWIN-254-M-1X16-VERTICAL") (at 109.22 33.02 0) (mirror y) (unit 1)
     (in_bom yes) (on_board yes)
     (property "Reference" "K1" (id 0) (at 109.22 30.48 0)
       (effects (font (size 1.15 1.15)))
     )
-    (property "Value" "GPIO IN" (id 1) (at 109.22 71.12 0)
-      (effects (font (size 1.15 1.15)))
-    )
-    (property "Footprint" "tronixio:HARWIN-M20-999154x" (id 2) (at 109.22 76.2 0)
-      (effects (font (size 1 1)) hide)
-    )
-    (property "Datasheet" "https://www.harwin.com/products/M20-9991546/" (id 3) (at 109.22 78.74 0)
-      (effects (font (size 1 1)) hide)
-    )
-    (property "Mouser" "855-M20-999154" (id 4) (at 109.22 81.28 0)
-      (effects (font (size 1 1)) hide)
-    )
-    (property "Name" "HARWIN-254-M-1X15-VERTICAL" (id 5) (at 109.22 73.66 0)
+    (property "Value" "GPIO IN" (id 1) (at 109.22 73.66 0)
+      (effects (font (size 1.15 1.15)))
+    )
+    (property "Footprint" "tronixio:HARWIN-M20-999164x" (id 2) (at 109.22 78.74 0)
+      (effects (font (size 1 1)) hide)
+    )
+    (property "Datasheet" "https://www.harwin.com/products/M20-9991646/" (id 3) (at 109.22 81.28 0)
+      (effects (font (size 1 1)) hide)
+    )
+    (property "Mouser" "855-M20-999164" (id 4) (at 109.22 83.82 0)
+      (effects (font (size 1 1)) hide)
+    )
+    (property "Name" "HARWIN-254-M-1X16-VERTICAL" (id 5) (at 109.22 76.2 0)
       (effects (font (size 1 1)) hide)
     )
@@
     (pin "14")
     (pin "15")
+    (pin "16")
     (pin "2")
     (pin "3")
@@
     (pin "6")
   )
-  (symbol (lib_id "tronixio:HARWIN-254-M-1X15-VERTICAL") (at 109.22 78.74 0) (mirror y) (unit 1)
+  (symbol (lib_id "tronixio:HARWIN-254-M-1X16-VERTICAL") (at 109.22 78.74 0) (mirror y) (unit 1)
     (in_bom yes) (on_board yes)
     (property "Reference" "K3" (id 0) (at 109.22 76.2 0)
       (effects (font (size 1.15 1.15)))
     )
-    (property "Value" "GPIO OUT #2" (id 1) (at 109.22 116.84 0)
-      (effects (font (size 1.15 1.15)))
-    )
-    (property "Footprint" "tronixio:HARWIN-M20-999154x" (id 2) (at 109.22 121.92 0)
-      (effects (font (size 1 1)) hide)
-    )
-    (property "Datasheet" "https://www.harwin.com/products/M20-9991546/" (id 3) (at 109.22 124.46 0)
-      (effects (font (size 1 1)) hide)
-    )
-    (property "Mouser" "855-M20-999154" (id 4) (at 109.22 127 0)
-      (effects (font (size 1 1)) hide)
-    )
-    (property "Name" "HARWIN-254-M-1X15-VERTICAL" (id 5) (at 109.22 119.38 0)
+    (property "Value" "GPIO OUT #2" (id 1) (at 109.22 119.38 0)
+      (effects (font (size 1.15 1.15)))
+    )
+    (property "Footprint" "tronixio:HARWIN-M20-999164x" (id 2) (at 109.22 124.46 0)
+      (effects (font (size 1 1)) hide)
+    )
+    (property "Datasheet" "https://www.harwin.com/products/M20-9991646/" (id 3) (at 109.22 127 0)
+      (effects (font (size 1 1)) hide)
+    )
+    (property "Mouser" "855-M20-999164" (id 4) (at 109.22 129.54 0)
+      (effects (font (size 1 1)) hide)
+    )
+    (property "Name" "HARWIN-254-M-1X16-VERTICAL" (id 5) (at 109.22 121.92 0)
       (effects (font (size 1 1)) hide)
     )
@@
     (pin "14")
     (pin "15")
+    (pin "16")
     (pin "2")
     (pin "3")
@@
     )
     (path "/9c4c3158-1d24-4d1c-8e39-342d19a63c17"
-      (reference "K1") (unit 1) (value "GPIO IN") (footprint "tronixio:HARWIN-M20-999154x")
+      (reference "K1") (unit 1) (value "GPIO IN") (footprint "tronixio:HARWIN-M20-999164x")
     )
     (path "/260fb712-9513-4ce5-b8a6-a42e234e006f"
-      (reference "K2") (unit 1) (value "GPIO OUT #1") (footprint "tronixio:HARWIN-M20-999154x")
+      (reference "K2") (unit 1) (value "GPIO OUT #1") (footprint "tronixio:HARWIN-M20-999164x")
     )
     (path "/a6f95181-d91e-4e5f-a676-e773e47b59e9"
-      (reference "K3") (unit 1) (value "GPIO OUT #2") (footprint "tronixio:HARWIN-M20-999154x")
+      (reference "K3") (unit 1) (value "GPIO OUT #2") (footprint "tronixio:HARWIN-M20-999164x")
     )
     (path "/a48ac013-6259-4020-bbba-a93d4f7fc8aa"
