File: Kicad/gpio-dg509b-header/dg509b.kicad_pcb (KiCad board)
At the start: 2 copper layers, 50 x 25 mm, 10 parts, among them K101 GPIO IN, K102 I/O, K103 I/O, U101 DG509BEY, U102 3M-SJ5376

Commit message: Update
Parts:
- removed C101: 100n, tronixio:CAPACITOR-SMD-1206
- removed K101: GPIO IN, tronixio:HARWIN-M20-975064x
- removed K102: I/O, tronixio:HARWIN-M20-999034x
- removed K103: I/O, tronixio:HARWIN-M20-999084x
- removed U101: DG509BEY, tronixio:SOIC-16
- removed U102: 3M-SJ5376, tronixio:3M-SJ5376
- added C1: 100n, tronixio:CAPACITOR-SMD-1206, F.Cu at (156.0, 63.5)
- added K1: GPIO IN, tronixio:HARWIN-M20-975064x, F.Cu at (169.8, 57.1)
- added K2: I/O, tronixio:HARWIN-M20-999034x, F.Cu at (146.5, 73.0)
- added K3: I/O, tronixio:HARWIN-M20-999084x, F.Cu at (127.0, 54.5)
- added R1: 10K, tronixio:RESISTOR-SMD-1206, F.Cu at (159.0, 63.5)
- added TP1: GND, tronixio:KEYSTONE-2000-3, F.Cu at (134.0, 72.0)
- added U1: DG509BEY, tronixio:SOIC-16, F.Cu at (149.0, 63.5)
- added U2: 3M-SJ5376, tronixio:3M-SJ5376, B.Cu at (134.0, 63.5)
- added kibuzzard-62B2FE4D: G***, kibuzzard-62B2FE4D, F.Cu at (149.0, 69.5)
- added kibuzzard-63494C1C: G***, kibuzzard-63494C1C, F.Cu at (137.5, 72.0)
- moved GT 24.0 mm to (149.0, 56.5)
- moved G*** 24.0 mm to (172.0, 73.5)
- moved kibuzzard-62B2FE3C 24.0 mm to (166.2, 57.1)
- moved kibuzzard-62B2FE4D 24.0 mm to (166.2, 59.7)
Routing:
- net Net-(K1-Pad3): track 0.00 -> 32.2 mm, vias 0 -> 1
- net Net-(K103-Pad1): track 26.5 -> 0.00 mm
- net Net-(K3-Pad1): track 0.00 -> 26.2 mm
- net Net-(K3-Pad5): track 0.00 -> 26.0 mm
- net Net-(K3-Pad6): track 0.00 -> 24.8 mm
- net Net-(K3-Pad2): track 0.00 -> 24.6 mm
- net Net-(K103-Pad8): track 24.0 -> 0.00 mm
- net Net-(K103-Pad2): track 24.0 -> 0.00 mm
- net Net-(K3-Pad7): track 0.00 -> 23.7 mm
- net Net-(K103-Pad5): track 23.3 -> 0.00 mm, vias 1 -> 0
- net Net-(K3-Pad3): track 0.00 -> 23.0 mm
- net VCC: track 6.36 -> 28.7 mm, vias 0 -> 1
- net Net-(K3-Pad8): track 0.00 -> 22.2 mm
- net Net-(K103-Pad6): track 22.1 -> 0.00 mm, vias 1 -> 0
- net Net-(K3-Pad4): track 0.00 -> 21.8 mm
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Other:
- board text added: "+20V"
- board text added: "30mA"
- board text added: "A0"
- board text added: "A1"
- board text added: "DA"
- board text added: "DB"
- board text added: "E"
- board text added: "GPIO - DG509B-HEADER - Rev.A - (01/2022) - Scale 100%"
- board text added: "S1A"
- board text added: "S1B"
- board text added: "S2A"
- board text added: "S2B"
- board text added: "S3A"
- board text added: "S3B"
- board text added: "S4A"
- board text added: "S4B"
- board text removed: "+2V/10V"
- board text removed: "1"
- board text removed: "1Y0"
- board text removed: "1Y1"
- board text removed: "1Z"
- board text removed: "2"
- board text removed: "2Y0"
- board text removed: "2Y1"
- board text removed: "2Z"
- board text removed: "3Y0"
- board text removed: "3Y1"
- board text removed: "3Z"
- board text removed: "5mA"
- board text removed: "GPIO - 74HC4053-HEADER - Rev.A - (01/2022) - Scale 100%"
- board text removed: "GPIO 74HC4053-HEADER"
- board text removed: "S1"
- board text removed: "S2"
- board text removed: "S3"
- board text removed: "~{E}"

Commit message: Up
Parts:
- moved TP1 1.00 mm to (135.0, 72.0)
- moved kibuzzard-63494C1C 1.00 mm to (138.5, 72.0)
Connections:
- net VCC renamed +VCC
