File: Kicad/gpio-dg509b-header/dg509b.kicad_pcb (KiCad board)
At the start: 2 copper layers, 50 x 25 mm, 14 parts, among them K1 GPIO IN, K2 I/O, K3 I/O, U1 DG509BEY, U2 3M-SJ5376

Commit message: Up
Parts:
- removed TP1: GND, tronixio:KEYSTONE-2000-3
- removed the kibuzzard-62B2FE4D at (149.0, 69.5)
- removed kibuzzard-63494C1C: G***, kibuzzard-63494C1C
- added C2: 100n, tronixio:CAPACITOR-SMD-1206, F.Cu at (156.0, 60.5)
- added K4: I/O, tronixio:HARWIN-M20-999084x, F.Cu at (127.0, 72.4)
- added kibuzzard-66858EC7: G***, kibuzzard-66858EC7, F.Cu at (145.2, 57.2)
- added kibuzzard-66858EE5: G***, kibuzzard-66858EE5, F.Cu at (150.3, 57.2)
- added kibuzzard-66858F0C: G***, kibuzzard-66858F0C, F.Cu at (152.8, 57.5)
- added kibuzzard-66858F12: G***, kibuzzard-66858F12, F.Cu at (147.8, 57.5)
- added kibuzzard-668593CE: G***, kibuzzard-668593CE, F.Cu at (149.0, 69.5)
- K3: value I/O -> VIN; footprint tronixio:HARWIN-M20-999084x -> tronixio:HARWIN-M20-999044x
- R1: value 10K -> 100k
- U1: value DG509BEY -> DG509B
- moved K3 25.8 mm to (152.8, 54.0), turned to -90 degrees
- moved C1 3.00 mm to (156.0, 66.5), turned to -90 degrees
- moved GT 2.00 mm to (149.0, 58.5)
Connections:
- C1 pad 1: +VCC -> V+
- C1 pad 2: GND -> POWER-GND
- K1 pad 1: +VCC -> POWER-+VCC
- K1 pad 2: GND -> POWER-GND
- K2 pad 1: Net-(U1-DA) -> Net-(U1-DB)
- K2 pad 2: GND -> POWER-GND
- K2 pad 3: Net-(U1-DB) -> Net-(U1-DA)
- K3 pad 1: Net-(K3-Pin_1) -> POWER-+VCC
- K3 pad 2: Net-(K3-Pin_2) -> V+
- K3 pad 3: Net-(K3-Pin_3) -> POWER-GND
- K3 pad 4: Net-(K3-Pin_4) -> V-
- R1 pad 2: GND -> POWER-GND
- U1 pad 10: Net-(K3-Pin_8) -> /S4B
- U1 pad 11: Net-(K3-Pin_7) -> /S3B
- U1 pad 12: Net-(K3-Pin_6) -> /S2B
- U1 pad 13: Net-(K3-Pin_5) -> /S1B
- U1 pad 14: +VCC -> V+
- U1 pad 15: GND -> POWER-GND
- U1 pad 3: GND -> V-
- U1 pad 4: Net-(K3-Pin_1) -> /S1A
- U1 pad 5: Net-(K3-Pin_2) -> /S2A
- U1 pad 6: Net-(K3-Pin_3) -> /S3A
- U1 pad 7: Net-(K3-Pin_4) -> /S4A
Routing:
- net +VCC: track 28.7 -> 0.00 mm, vias 1 -> 0
- net Net-(K3-Pin_1): track 26.2 -> 0.00 mm
- net /S1A: track 0.00 -> 26.1 mm
- net Net-(K3-Pin_5): track 26.0 -> 0.00 mm
- net /S1B: track 0.00 -> 25.7 mm
- net Net-(K3-Pin_6): track 24.8 -> 0.00 mm
- net Net-(K3-Pin_2): track 24.6 -> 0.00 mm
- net /S2B: track 0.00 -> 24.5 mm
- net /S2A: track 0.00 -> 23.7 mm
- net Net-(K3-Pin_7): track 23.7 -> 0.00 mm
- net /S3B: track 0.00 -> 23.2 mm
- net Net-(K3-Pin_3): track 23.0 -> 0.00 mm
- net /S4B: track 0.00 -> 22.5 mm
- net Net-(K3-Pin_8): track 22.2 -> 0.00 mm
- net /S3A: track 0.00 -> 21.8 mm
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- added copper zone on B.Cu, net POWER-GND
- removed copper zone on B.Cu, net GND
