File: Kicad/gpio-dg509b-header/dg509b.kicad_sch (KiCad schematic)
At the start: 6 parts, among them K101 GPIO IN, K102 I/O, K103 I/O, U101 DG509BEY, U102 3M-SJ5376

Commit message: Update
Parts:
- added R1: 10K, tronixio:RESISTOR-SMD-1206, symbol tronixio:RESISTOR-1206-10K
- added TP1: GND, tronixio:KEYSTONE-2000-3, symbol tronixio:KEYSTONE-2000-3
- renumbered C101 to C1, K101 to K1, K102 to K2, K103 to K3, U101 to U1, U102 to U2
Connections:
- net GND: now also R1.2, TP1.1
- net at K1.3, U1.2 (E): now also R1.1
Other:
- moved on the sheet: K1, K2

Commit message: Up
Parts:
- C1: symbol tronixio:CAPACITOR-1206-100N -> tronixio:CAPACITOR-1206-100N-50V-5P-X7R; Mouser 80-C1206C104M5R -> 80-C1206C104J5R; Name CAPACITOR-1206-100N -> (none); Tolerance 20% -> 5%
- K1: Name HARWIN-254-M-1X06-RIGHT-ANGLE -> (none)
- K2: Name HARWIN-254-M-1X03-VERTICAL -> (none)
- K3: Name HARWIN-254-M-1X08-VERTICAL -> (none)
- R1: symbol tronixio:RESISTOR-1206-10K -> tronixio:RESISTOR-1206-10K-5P; Name RESISTOR-1206-10K -> (none)
- TP1: Name KEYSTONE-2000-3 -> (none)
- U1: symbol tronixio:VISHAY-DG509BEY-SOIC-16 -> tronixio:VISHAY-DG509BEY-SOIC; Name VISHAY-DG509BEY-SOIC-16 -> (none)
Connections:
- net VCC renamed +VCC
Other:
- moved on the sheet: C1, K3, R1, U1
