File: Kicad/gpio-dg509b-header/dg509b.kicad_sch (KiCad schematic)
At the start: 8 parts, among them K1 GPIO IN, K2 I/O, K3 I/O, U1 DG509BEY, U2 3M-SJ5376

Commit message: Up
Parts:
- removed TP1: GND, tronixio:KEYSTONE-2000-3, symbol tronixio:KEYSTONE-2000-3
- added C2: 100n, tronixio:CAPACITOR-SMD-1206, symbol tronixio:CAPACITOR-1206-100N-50V-5P-X7R
- added K3: VIN, tronixio:HARWIN-M20-999044x, symbol tronixio:HARWIN-254-M-1X04-VERTICAL
- R1: value 10K -> 100k; symbol tronixio:RESISTOR-1206-10K-5P -> tronixio:RESISTOR-1206-100K-5P; Mouser 660-RK73B2BTTDD103J -> 660-RK73B2BTTDD104J
- U1: value DG509BEY -> DG509B; symbol tronixio:VISHAY-DG509BEY-SOIC -> tronixio:VISHAY-DG509B-SOIC
- renumbered K3 to K4
Connections:
- net POWER-GND: now also C2.2, K3.3; no longer U1.3 (V-)
- net at K2.1: now also U1.9 (DB); no longer U1.8 (DA)
- net at K2.3: now also U1.8 (DA); no longer U1.9 (DB)
- net S1A: now reaches U1.4 (S1A)
- net S1A: now also K4.8 (Pin_8); no longer K4.1 (Pin_1)
- net S2A: now reaches U1.5 (S2A)
- net S2A: now also K4.7 (Pin_7); no longer K4.2 (Pin_2)
- net S2B: now reaches K4.3 (Pin_3)
- net S2B: now also U1.12 (S2B); no longer U1.6 (S3A)
- net S1B: now reaches K4.4 (Pin_4)
- net S1B: now also U1.13 (S1B); no longer U1.7 (S4A)
- net S4A: now reaches K4.5 (Pin_5)
- net S4A: now also U1.7 (S4A); no longer U1.13 (S1B)
- net S3A: now reaches K4.6 (Pin_6)
- net S3A: now also U1.6 (S3A); no longer U1.12 (S2B)
- net S3B: now reaches U1.11 (S3B)
- net S3B: now also K4.2 (Pin_2); no longer K4.7 (Pin_7)
- net S4B: now reaches U1.10 (S4B)
- net S4B: now also K4.1 (Pin_1); no longer K4.8 (Pin_8)
- net POWER-VBAT renamed V+
- net V+: now also K3.2; no longer K1.1
- new net POWER-+VCC: K1.1, K3.1
- new net V-: C2.1, K3.4, U1.3 (V-)
Other:
- note removed: "~{E}"
- moved on the sheet: C1, K1, K2, K4, R1, U1
