File: Kicad/gpio-dg509b-header/main.kicad_pcb (KiCad board)
At the start: 2 copper layers, 50 x 25 mm, 18 parts, among them K1 GPIO IN, K2 I/O, K3 VIN, K4 I/O, U1 DG509B, U2 3M-SJ5376

Commit message: Up
Other:
- board text added: "2022Q1 - Rev.A"
- board text added: "GPIO - DG509B-HEADER - Rev.A - (Q1/2022) - Scale 100%"
- board text added: "±20V"
- board text removed: "+20V"
- board text removed: "202201 - Rev.A"
- board text removed: "GPIO - DG509B-HEADER - Rev.A - (01/2022) - Scale 100%"
Changed lines of the file:
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@@
 	(title_block
 		(title "GPIO - DG509B-HEADER")
-		(date "01/2022")
+		(date "Q1/2022")
 		(rev "A")
 	)
@@
 			)
 		)
-		(property "Footprint" ""
+		(property "Footprint" "tronixio:OSHW-3MM"
 			(at 0 0 0)
 			(unlocked yes)
@@
 				(font
 					(size 0.001 0.001)
+					(thickness 0.15)
 				)
 			)
@@
 				(font
 					(size 0.001 0.001)
+					(thickness 0.15)
 				)
 			)
@@
 		)
 		(sheetname "Root")
-		(sheetfile "dg509b.kicad_sch")
+		(sheetfile "main.kicad_sch")
 		(attr through_hole)
 		(fp_line
@@
 		)
 		(sheetname "Root")
-		(sheetfile "dg509b.kicad_sch")
+		(sheetfile "main.kicad_sch")
 		(attr through_hole)
 		(fp_line
@@
 		(at 127 72.39 180)
 		(property "Reference" "K4"
-			(at 0 20 360)
+			(at 0 20 0)
 			(layer "F.SilkS")
 			(hide yes)
@@
 		)
 		(property "Footprint" "tronixio:HARWIN-M20-999084x"
-			(at 0 0 360)
+			(at 0 0 0)
 			(layer "F.Fab")
 			(hide yes)
@@
 		)
 		(property "Datasheet" "https://www.harwin.com/products/M20-9990846/"
-			(at 0 0 360)
+			(at 0 0 0)
 			(layer "F.Fab")
 			(hide yes)
@@
 		)
 		(property "Description" "M20 Series - 2.54mm Pitch PCB Connector"
-			(at 0 0 360)
+			(at 0 0 0)
 			(layer "F.Fab")
 			(hide yes)
@@
 		)
 		(sheetname "Root")
-		(sheetfile "dg509b.kicad_sch")
+		(sheetfile "main.kicad_sch")
 		(attr through_hole)
 		(fp_line
@@
 				(font
 					(size 0.001 0.001)
+					(thickness 0.15)
 				)
 			)
@@
 				(font
 					(size 0.001 0.001)
+					(thickness 0.15)
 				)
 			)
@@
 		)
 		(sheetname "Root")
-		(sheetfile "dg509b.kicad_sch")
+		(sheetfile "main.kicad_sch")
 		(attr smd)
 		(fp_line
@@
 			(end 1.5 4.5)
 			(stroke
-				(width 0.15)
+				(width 0.2)
 				(type solid)
 			)
@@
 			(end 1.5 -4.5)
 			(stroke
-				(width 0.15)
+				(width 0.2)
 				(type solid)
 			)
@@
 			(end -1.5 4.5)
 			(stroke
-				(width 0.15)
+				(width 0.2)
 				(type solid)
 			)
@@
 			(end -1.5 -4.5)
 			(stroke
-				(width 0.15)
+				(width 0.2)
 				(type solid)
 			)
@@
 			(end 0.5 -4.5)
 			(stroke
-				(width 0.15)
+				(width 0.2)
 				(type solid)
 			)
@@
 			(end -0.5 -4.5)
 			(stroke
-				(width 0.15)
+				(width 0.2)
 				(type solid)
 			)
@@
 				(font
 					(size 0.001 0.001)
+					(thickness 0.15)
 				)
 			)
@@
 				(font
 					(size 0.001 0.001)
+					(thickness 0.15)
 				)
 			)
@@
 		)
 		(sheetname "Root")
-		(sheetfile "dg509b.kicad_sch")
+		(sheetfile "main.kicad_sch")
 		(attr smd)
 		(fp_line
@@
 				(font
 					(size 0.001 0.001)
+					(thickness 0.15)
 				)
 			)
@@
 				(font
 					(size 0.001 0.001)
+					(thickness 0.15)
 				)
 			)
@@
 		)
 		(sheetname "Root")
-		(sheetfile "dg509b.kicad_sch")
+		(sheetfile "main.kicad_sch")
 		(attr through_hole)
 		(fp_line
@@
 		)
 		(sheetname "Root")
-		(sheetfile "dg509b.kicad_sch")
+		(sheetfile "main.kicad_sch")
 		(attr smd)
 		(fp_line
@@
 		)
 		(sheetname "Root")
-		(sheetfile "dg509b.kicad_sch")
+		(sheetfile "main.kicad_sch")
 		(attr smd)
 		(fp_line
@@
 				(font
 					(size 0.001 0.001)
+					(thickness 0.15)
 				)
 			)
@@
 				(font
 					(size 0.001 0.001)
+					(thickness 0.15)
 				)
 			)
@@
 			)
 		)
-		(property "Footprint" ""
+		(property "Footprint" "tronixio:OSHW-5MM"
 			(at 0 0 180)
 			(unlocked yes)
@@
 		)
 		(sheetname "Root")
-		(sheetfile "dg509b.kicad_sch")
+		(sheetfile "main.kicad_sch")
 		(zone_connect 0)
 		(fp_circle
@@
 			(end 4.2 0)
 			(stroke
-				(width 0.15)
+				(width 0.2)
 				(type solid)
 			)
@@
 		)
 	)
-	(gr_text "202201 - Rev.A"
+	(gr_text "2022Q1 - Rev.A"
 		(at 149 69.572893 0)
 		(layer "B.SilkS")
@@
 		)
 	)
-	(gr_text "202201 - Rev.A"
+	(gr_text "2022Q1 - Rev.A"
 		(at 125.5 74.75 0)
 		(layer "F.SilkS")
@@
 		)
 	)
-	(gr_text "+20V"
+	(gr_text "±20V"
 		(at 173.5 52.5 0)
 		(layer "F.SilkS")
@@
 		)
 	)
-	(gr_text "GPIO - DG509B-HEADER - Rev.A - (01/2022) - Scale 100%"
+	(gr_text "GPIO - DG509B-HEADER - Rev.A - (Q1/2022) - Scale 100%"
 		(at 124 86 0)
 		(layer "Dwgs.User")
