File: Kicad/gpio-hc4053-header/hc4053-header.kicad_pcb (KiCad board)
At the start: 2 copper layers, 50 x 25 mm, 10 parts, among them K1 GPIO IN, K3 I/O, K4 I/O, U1 74HC4053, U2 3M-SJ5376

Commit message: Update
Other:
- board text removed: "Q0"
- board text removed: "Q1"
- board text removed: "Q2"
- board text removed: "Q3"
- board text removed: "Q4"
- board text removed: "Q5"
- board text removed: "Q6"
- board text removed: "Q7"
Changed lines of the file:
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@@
     (effects (font (size 1 1) (thickness 0.15)) (justify right))
-  )
-  (gr_text "Q4" (at 141.62 79) (layer "F.SilkS")
-    (effects (font (size 1 1) (thickness 0.15)))
-  )
-  (gr_text "Q2" (at 125.92 79) (layer "F.SilkS")
-    (effects (font (size 1 1) (thickness 0.15)))
   )
   (gr_text "~{E}" (at 144 69.85) (layer "F.SilkS")
@@
     (effects (font (size 1 1) (thickness 0.15)) (justify right))
   )
-  (gr_text "JLCJLCJLCJLC" (at 107 79) (layer "F.SilkS")
+  (gr_text "JLCJLCJLCJLC" (at 148 63.5 90) (layer "F.SilkS")
     (effects (font (size 0.8 0.8) (thickness 0.1)))
-  )
-  (gr_text "Q0" (at 151.78 79) (layer "F.SilkS")
-    (effects (font (size 1 1) (thickness 0.15)))
   )
   (gr_text "2Y1" (at 104.75 57.15) (layer "F.SilkS")
@@
     (effects (font (size 1 1) (thickness 0.15)))
   )
-  (gr_text "Q1" (at 128.46 79) (layer "F.SilkS")
-    (effects (font (size 1 1) (thickness 0.15)))
-  )
   (gr_text "3Y1" (at 104.75 62.23) (layer "F.SilkS")
     (effects (font (size 1 1) (thickness 0.15)) (justify left))
-  )
-  (gr_text "Q7" (at 134 79) (layer "F.SilkS")
-    (effects (font (size 1 1) (thickness 0.15)))
   )
   (gr_text "202201 - Rev.A" (at 100.5 74.5) (layer "F.SilkS")
@@
     (effects (font (size 1 1) (thickness 0.15)) (justify right))
   )
-  (gr_text "Q4" (at 120.84 79) (layer "F.SilkS")
-    (effects (font (size 1 1) (thickness 0.15)))
-  )
   (gr_text "GPIO 74HC4053-HEADER" (at 100.5 72.5) (layer "F.SilkS")
     (effects (font (size 1 1) (thickness 0.2)) (justify left))
-  )
-  (gr_text "Q7" (at 113.22 79) (layer "F.SilkS")
-    (effects (font (size 1 1) (thickness 0.15)))
   )
   (gr_text "1Y1" (at 104.75 67.31) (layer "F.SilkS")
@@
   (gr_text "S2" (at 144 64.77) (layer "F.SilkS")
     (effects (font (size 1 1) (thickness 0.15)) (justify right))
-  )
-  (gr_text "Q6" (at 136.54 79) (layer "F.SilkS")
-    (effects (font (size 1 1) (thickness 0.15)))
   )
   (gr_text "www.tronix.io" (at 146 72.5) (layer "F.SilkS")
@@
     (effects (font (size 1 1) (thickness 0.15)) (justify right))
   )
-  (gr_text "Q1" (at 149.24 79) (layer "F.SilkS")
-    (effects (font (size 1 1) (thickness 0.15)))
-  )
   (gr_text "1Y0" (at 104.75 69.85) (layer "F.SilkS")
     (effects (font (size 1 1) (thickness 0.15)) (justify left))
-  )
-  (gr_text "Q2" (at 146.7 79) (layer "F.SilkS")
-    (effects (font (size 1 1) (thickness 0.15)))
-  )
-  (gr_text "Q5" (at 139.08 79) (layer "F.SilkS")
-    (effects (font (size 1 1) (thickness 0.15)))
-  )
-  (gr_text "Q5" (at 118.3 79) (layer "F.SilkS")
-    (effects (font (size 1 1) (thickness 0.15)))
   )
   (gr_text "5mA" (at 149.5 54.5) (layer "F.SilkS")
     (effects (font (size 1 1) (thickness 0.15)) (justify right))
   )
-  (gr_text "Q0" (at 131 79) (layer "F.SilkS")
-    (effects (font (size 1 1) (thickness 0.15)))
-  )
-  (gr_text "Q6" (at 115.76 79) (layer "F.SilkS")
-    (effects (font (size 1 1) (thickness 0.15)))
-  )
-  (gr_text "Q3" (at 123.38 79) (layer "F.SilkS")
-    (effects (font (size 1 1) (thickness 0.15)))
-  )
-  (gr_text "Q3" (at 144.16 79) (layer "F.SilkS")
-    (effects (font (size 1 1) (thickness 0.15)))
-  )
   (gr_text "GPIO 74HC4053-HEADER - Rev.A - (01/2022) - Scale 100%" (at 100 86) (layer "Dwgs.User")

Commit message: Update
Parts:
- U2: footprint tronixio:zzz3M-SJ5376 -> tronixio:3M-SJ5376
Connections:
- K4 pad 1: Net-(U1-Pad1) -> Net-(U1-Pad12)
- K4 pad 2: Net-(U1-Pad2) -> Net-(U1-Pad13)
- K4 pad 3: Net-(U1-Pad3) -> Net-(U1-Pad2)
- K4 pad 4: Net-(U1-Pad5) -> Net-(U1-Pad1)
- K4 pad 5: Net-(U1-Pad13) -> Net-(U1-Pad5)
- K4 pad 6: Net-(U1-Pad12) -> Net-(U1-Pad3)
Routing:
- net Net-(K3-Pad2): track 20.3 -> 0.00 mm, vias 1 -> 0
- net Net-(K3-Pad1): track 20.1 -> 0.00 mm, vias 1 -> 0
- net Net-(K1-Pad6): track 32.6 -> 28.7 mm, vias 0 -> 1
- net Net-(U1-Pad1): track 19.2 -> 22.4 mm, vias 0 -> 1
- net Net-(U1-Pad3): track 20.3 -> 23.5 mm, vias 0 -> 1
- net Net-(U1-Pad12): track 31.4 -> 33.9 mm
- net Net-(U1-Pad5): track 20.3 -> 21.4 mm
- net Net-(U1-Pad2): track 19.8 -> 20.8 mm
- net Net-(U1-Pad13): track 30.9 -> 31.8 mm
- net GND: track 4.59 -> 4.04 mm, vias 1 -> 0
Other:
- outline, holes or cut-outs redrawn
- board text added: "GPIO - 74HC4053-HEADER - Rev.A - (01/2022) - Scale 100%"
- board text removed: "GPIO 74HC4053-HEADER - Rev.A - (01/2022) - Scale 100%"

Commit message: Update
Parts:
- C1: footprint tronixio:CAPACITOR-1206 -> tronixio:CAPACITOR-SMD-1206
Routing:
- net Net-(K3-Pad2): track 0.00 -> 22.4 mm, vias 0 -> 1
- net Net-(K3-Pad1): track 0.00 -> 22.2 mm, vias 0 -> 1
- net Net-(K1-Pad6): track 28.7 -> 32.1 mm, vias 1 -> 0
- net Net-(K4-Pad2): track 31.8 -> 29.8 mm
- net Net-(K3-Pad3): track 15.5 -> 14.4 mm
- net GND: track 4.04 -> 4.48 mm, vias 0 -> 1

Commit message: Update
Parts:
- removed K4: I/O, tronixio:HARWIN-M20-999064x
- added K2: I/O, tronixio:HARWIN-M20-999034x, F.Cu at (152.0, 73.0)
- added TP1: GND, tronixio:KEYSTONE-2000-3, F.Cu at (137.0, 54.0)
- added kibuzzard-63494430: G***, kibuzzard-63494430, F.Cu at (140.5, 54.0)
- K3: footprint tronixio:HARWIN-M20-999034x -> tronixio:HARWIN-M20-999064x
- moved U1 24.5 mm to (149.5, 61.5)
- moved C1 24.5 mm to (149.5, 68.0)
- moved G*** 24.5 mm to (172.5, 73.5)
- moved GT 24.5 mm to (149.5, 57.0)
- moved K1 24.5 mm to (170.3, 57.1)
- moved kibuzzard-62B2FE3C 24.5 mm to (166.8, 57.1)
- moved kibuzzard-62B2FE4D 24.5 mm to (166.8, 59.7)
- moved U2 22.5 mm to (134.5, 63.5)
- moved K3 15.9 mm to (127.5, 57.1), turned to 0 degrees
Connections:
- U1 pad 1: Net-(K4-Pad4) -> Net-(K3-Pad4)
- U1 pad 12: Net-(K4-Pad1) -> Net-(K3-Pad1)
- U1 pad 13: Net-(K4-Pad2) -> Net-(K3-Pad2)
- U1 pad 14: Net-(K3-Pad1) -> Net-(K2-Pad1)
- U1 pad 15: Net-(K3-Pad2) -> Net-(K2-Pad2)
- U1 pad 2: Net-(K4-Pad3) -> Net-(K3-Pad3)
- U1 pad 3: Net-(K4-Pad6) -> Net-(K3-Pad6)
- U1 pad 4: Net-(K3-Pad3) -> Net-(K2-Pad3)
- U1 pad 5: Net-(K4-Pad5) -> Net-(K3-Pad5)
Routing:
- net Net-(K4-Pad1): track 34.4 -> 0.00 mm, vias 1 -> 0
- net Net-(K4-Pad2): track 29.8 -> 0.00 mm, vias 1 -> 0
- net Net-(K3-Pad6): track 0.00 -> 23.5 mm, vias 0 -> 1
- net Net-(K4-Pad6): track 23.5 -> 0.00 mm, vias 1 -> 0
- net Net-(K2-Pad2): track 0.00 -> 22.5 mm, vias 0 -> 1
- net Net-(K3-Pad4): track 0.00 -> 22.4 mm, vias 0 -> 1
- net Net-(K4-Pad4): track 22.4 -> 0.00 mm, vias 1 -> 0
- net Net-(K2-Pad1): track 0.00 -> 22.3 mm, vias 0 -> 1
- net Net-(K3-Pad5): track 0.00 -> 21.4 mm
- net Net-(K4-Pad5): track 21.4 -> 0.00 mm
- net Net-(K4-Pad3): track 20.8 -> 0.00 mm
- net Net-(K2-Pad3): track 0.00 -> 14.5 mm, vias 0 -> 1
- net Net-(K3-Pad1): track 22.2 -> 34.3 mm
- net Net-(K3-Pad2): track 22.4 -> 29.7 mm
- net Net-(K3-Pad3): track 14.4 -> 20.9 mm, vias 1 -> 0
Other:
- board text added: "+5V"
- board text added: "50mA"
- board text removed: "+2V/10V"
- board text removed: "5mA"

Commit message: Update
Parts:
- added C2: 100n, tronixio:CAPACITOR-SMD-1206, F.Cu at (149.5, 68.0)
- added R1: 10K, tronixio:RESISTOR-SMD-1206, F.Cu at (141.0, 65.5)
- C1: value 100n -> 10n
- moved C1 6.50 mm to (143.5, 65.5), turned to -90 degrees
- moved GT 0.50 mm to (149.5, 56.5)
Connections:
- C1 pad 1: VCC -> Net-(C1-Pad1)
- K1 pad 6: Net-(K1-Pad6) -> Net-(C1-Pad1)
- U1 pad 6: Net-(K1-Pad6) -> Net-(C1-Pad1)
Routing:
- net Net-(C1-Pad1): track 0.00 -> 39.5 mm, vias 0 -> 2
- net Net-(K1-Pad6): track 32.2 -> 0.00 mm
- net VCC: track 30.6 -> 43.5 mm
- net GND: track 4.58 -> 8.24 mm
Other:
- board text added: "+2V/+10V"
- board text removed: "+5V"
