File: Kicad/gpio-hc4053-header/hc4053-header.kicad_pcb (KiCad board)
At the start: 2 copper layers, 50 x 25 mm, 14 parts, among them K1 GPIO IN, K2 I/O, K3 I/O, U1 74HC4053, U2 3M-SJ5376

Commit message: GPIO HC4053
Parts:
- R1: value 10K -> 10k
- moved K1 24.0 mm to (170.8, 81.2)
- moved K3 24.0 mm to (128.0, 81.2)
- moved kibuzzard-62B2FE3C 24.0 mm to (167.2, 81.2)
- moved C1 24.0 mm to (144.0, 89.5)
- moved C2 24.0 mm to (150.0, 92.0)
- moved G*** 24.0 mm to (173.0, 97.5)
- moved GT 24.0 mm to (150.0, 80.5)
- moved K2 24.0 mm to (152.5, 97.0)
- moved R1 24.0 mm to (141.5, 89.5)
- moved TP1 24.0 mm to (137.5, 78.0)
- moved U1 24.0 mm to (150.0, 85.5)
- moved U2 24.0 mm to (135.0, 87.5)
- moved kibuzzard-62B2FE4D 24.0 mm to (167.2, 83.7)
- moved kibuzzard-63494430 24.0 mm to (141.0, 78.0)
Connections:
- net VCC renamed +VCC
Other:
- board text added: "5mA"
- board text removed: "50mA"
