File: Kicad/gpio-hc4053-header/hc4053-header.kicad_sch (KiCad schematic)
At the start: 6 parts, among them K1 GPIO IN, K3 I/O, K4 I/O, U1 74HC4053, U2 3M-SJ5376

Commit message: Update
Parts:
- C1: symbol tronixio:C-1206 -> tronixio:CAPACITOR-1206-100N; Mouser (none) -> 80-C1206C104M5R; Name (none) -> CAPACITOR-1206-100N; Tolerance (none) -> 20%; Voltage (none) -> 50V
- K1: Name (none) -> HARWIN-254-M-1X06-RIGHT-ANGLE
- K3: Name (none) -> HARWIN-254-M-1X03-VERTICAL
- K4: Name (none) -> HARWIN-254-M-1X06-VERTICAL
- U1: symbol tronixio:74HC4053 -> tronixio:74HC4053-SOIC-16; Name (none) -> 74HC4053-SOIC-16
- U2: footprint tronixio:zzz3M-SJ5376 -> tronixio:3M-SJ5376
Connections:
- net at K4.1: now also U1.12 (1Y0); no longer U1.1 (2Y1)
- net at K4.2: now also U1.13 (1Y1); no longer U1.2 (2Y0)
- net at K4.3: now also U1.2 (2Y0); no longer U1.3 (3Y1)
- net at K4.4: now also U1.1 (2Y1); no longer U1.5 (3Y0)
- net at K4.5: now also U1.5 (3Y0); no longer U1.13 (1Y1)
- net at K4.6: now also U1.3 (3Y1); no longer U1.12 (1Y0)
Other:
- moved on the sheet: C1, K1, K3, K4, U1

Commit message: Update
Parts:
- C1: footprint tronixio:CAPACITOR-1206 -> tronixio:CAPACITOR-SMD-1206
Other:
- moved on the sheet: C1, K1, K3, K4, U1

Commit message: Update
Parts:
- added TP1: GND, tronixio:KEYSTONE-2000-3, symbol tronixio:KEYSTONE-2000-3
- renumbered K3 to K2, K4 to K3
Connections:
- net GND: now also TP1.1
Changed lines of the file:
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@@
     (stroke (width 0) (type default) (color 0 0 0 0))
+  )
+  (wire (pts (xy 162.56 185.42) (xy 162.56 190.5))
+    (stroke (width 0) (type solid) (color 0 0 0 0))
   )
   (wire (pts (xy 162.56 68.58) (xy 165.1 68.58))
@@
   (symbol (lib_id "tronixio:HARWIN-254-M-1X03-VERTICAL") (at 111.76 86.36 0) (mirror y) (unit 1)
     (in_bom yes) (on_board yes)
-    (property "Reference" "K3" (id 0) (at 111.76 96.52 0)
-      (effects (font (size 1.15 1.15)))
-    )
-    (property "Value" "I/O" (id 1) (at 111.76 93.98 0)
+    (property "Reference" "K2" (id 0) (at 111.76 93.98 0)
+      (effects (font (size 1.15 1.15)))
+    )
+    (property "Value" "I/O" (id 1) (at 111.76 96.52 0)
       (effects (font (size 1.15 1.15)))
     )
@@
   (symbol (lib_id "tronixio:HARWIN-254-M-1X06-VERTICAL") (at 182.88 76.2 0) (unit 1)
     (in_bom yes) (on_board yes)
-    (property "Reference" "K4" (id 0) (at 181.61 73.66 0)
-      (effects (font (size 1.15 1.15)) (justify left))
+    (property "Reference" "K3" (id 0) (at 182.88 73.66 0)
+      (effects (font (size 1.15 1.15)))
     )
     (property "Value" "I/O" (id 1) (at 182.88 91.44 0)
@@
   (symbol (lib_id "tronixio:POWER-VCC") (at 129.54 60.96 0) (unit 1)
     (in_bom yes) (on_board yes)
-    (property "Reference" "#PWR03" (id 0) (at 134.62 58.42 0)
+    (property "Reference" "#PWR0103" (id 0) (at 134.62 58.42 0)
       (effects (font (size 1 1)) hide)
     )
@@
   (symbol (lib_id "tronixio:POWER-FLAG") (at 177.8 190.5 180) (unit 1)
     (in_bom yes) (on_board yes) (fields_autoplaced)
-    (property "Reference" "#FLG02" (id 0) (at 177.8 188.595 0)
+    (property "Reference" "#FLG0102" (id 0) (at 177.8 188.595 0)
       (effects (font (size 1.27 1.27)) hide)
     )
@@
     (pin "6")
   )
+  (symbol (lib_id "tronixio:POWER-GND") (at 162.56 190.5 0) (unit 1)
+    (in_bom yes) (on_board yes)
+    (property "Reference" "#PWR0106" (id 0) (at 162.56 195.58 0)
+      (effects (font (size 1 1)) hide)
+    )
+    (property "Value" "POWER-GND" (id 1) (at 162.56 198.12 0)
+      (effects (font (size 1 1)) hide)
+    )
+    (property "Footprint" "" (id 2) (at 162.56 190.5 0)
+      (effects (font (size 1 1)) hide)
+    )
+    (property "Datasheet" "" (id 3) (at 162.56 190.5 0)
+      (effects (font (size 1 1)) hide)
+    )
+    (pin "1")
+  )
   (symbol (lib_id "tronixio:POWER-VCC") (at 116.84 60.96 0) (unit 1)
     (in_bom yes) (on_board yes)
-    (property "Reference" "#PWR02" (id 0) (at 121.92 58.42 0)
+    (property "Reference" "#PWR0101" (id 0) (at 121.92 58.42 0)
       (effects (font (size 1 1)) hide)
     )
@@
   (symbol (lib_id "tronixio:POWER-GND") (at 134.62 106.68 0) (unit 1)
     (in_bom yes) (on_board yes)
-    (property "Reference" "#PWR05" (id 0) (at 134.62 111.76 0)
+    (property "Reference" "#PWR0105" (id 0) (at 134.62 111.76 0)
       (effects (font (size 1 1)) hide)
     )
@@
   (symbol (lib_id "tronixio:POWER-GND") (at 170.18 190.5 0) (unit 1)
     (in_bom yes) (on_board yes)
-    (property "Reference" "#PWR06" (id 0) (at 170.18 195.58 0)
+    (property "Reference" "#PWR0108" (id 0) (at 170.18 195.58 0)
       (effects (font (size 1 1)) hide)
     )
@@
     (pin "1")
   )
+  (symbol (lib_id "tronixio:KEYSTONE-2000-3") (at 162.56 185.42 0) (unit 1)
+    (in_bom yes) (on_board yes)
+    (property "Reference" "TP1" (id 0) (at 162.56 180.34 0)
+      (effects (font (size 1.15 1.15)))
+    )
+    (property "Value" "GND" (id 1) (at 165.1 184.1499 0)
+      (effects (font (size 1.15 1.15)) (justify left) hide)
+    )
+    (property "Footprint" "tronixio:KEYSTONE-2000-3" (id 2) (at 162.56 195.58 0)
+      (effects (font (size 1 1)) hide)
+    )
+    (property "Datasheet" "https://www.keyelco.com/product.cfm/product_id/3037" (id 3) (at 162.56 198.12 0)
+      (effects (font (size 1 1)) hide)
+    )
+    (property "Name" "KEYSTONE-2000-3" (id 4) (at 162.56 193.04 0)
+      (effects (font (size 1 1)) hide)
+    )
+    (property "Mouser" "534-2000-3" (id 5) (at 162.56 200.66 0)
+      (effects (font (size 1 1)) hide)
+    )
+    (pin "1")
+  )
   (symbol (lib_id "tronixio:POWER-GND") (at 129.54 106.68 0) (unit 1)
     (in_bom yes) (on_board yes)
-    (property "Reference" "#PWR04" (id 0) (at 129.54 111.76 0)
+    (property "Reference" "#PWR0104" (id 0) (at 129.54 111.76 0)
       (effects (font (size 1 1)) hide)
     )
@@
   (symbol (lib_id "tronixio:POWER-GND") (at 165.1 106.68 0) (unit 1)
     (in_bom yes) (on_board yes)
-    (property "Reference" "#PWR0101" (id 0) (at 165.1 111.76 0)
+    (property "Reference" "#PWR0107" (id 0) (at 165.1 111.76 0)
       (effects (font (size 1 1)) hide)
     )
@@
   (symbol (lib_id "tronixio:POWER-GND") (at 116.84 106.68 0) (unit 1)
     (in_bom yes) (on_board yes)
-    (property "Reference" "#PWR01" (id 0) (at 116.84 111.76 0)
+    (property "Reference" "#PWR0102" (id 0) (at 116.84 111.76 0)
       (effects (font (size 1 1)) hide)
     )
@@
   (symbol (lib_id "tronixio:POWER-FLAG") (at 170.18 185.42 0) (unit 1)
     (in_bom yes) (on_board yes) (fields_autoplaced)
-    (property "Reference" "#FLG01" (id 0) (at 170.18 187.325 0)
+    (property "Reference" "#FLG0101" (id 0) (at 170.18 187.325 0)
       (effects (font (size 1.27 1.27)) hide)
     )
@@
   (symbol (lib_id "tronixio:POWER-VCC") (at 177.8 185.42 0) (unit 1)
     (in_bom yes) (on_board yes)
-    (property "Reference" "#PWR07" (id 0) (at 182.88 182.88 0)
+    (property "Reference" "#PWR0109" (id 0) (at 182.88 182.88 0)
       (effects (font (size 1 1)) hide)
     )
@@
   (symbol_instances
     (path "/fc217884-314f-464c-b6f5-43d868b35e41"
-      (reference "#FLG01") (unit 1) (value "PWR_FLAG") (footprint "")
+      (reference "#FLG0101") (unit 1) (value "PWR_FLAG") (footprint "")
     )
     (path "/9702bc62-2308-42c6-8752-e186afd16157"
-      (reference "#FLG02") (unit 1) (value "PWR_FLAG") (footprint "")
+      (reference "#FLG0102") (unit 1) (value "PWR_FLAG") (footprint "")
+    )
+    (path "/baf11eeb-f067-4869-87da-54cc7a8dad87"
+      (reference "#PWR0101") (unit 1) (value "POWER-VBAT") (footprint "")
     )
     (path "/eb2937d0-b93f-40a9-8c3e-0dc385a8c8af"
-      (reference "#PWR01") (unit 1) (value "POWER-GND") (footprint "")
-    )
-    (path "/baf11eeb-f067-4869-87da-54cc7a8dad87"
-      (reference "#PWR02") (unit 1) (value "POWER-VBAT") (footprint "")
+      (reference "#PWR0102") (unit 1) (value "POWER-GND") (footprint "")
     )
     (path "/5d92ba57-17d7-429e-bdc9-e4bb7cabea57"
-      (reference "#PWR03") (unit 1) (value "POWER-VBAT") (footprint "")
+      (reference "#PWR0103") (unit 1) (value "POWER-VBAT") (footprint "")
     )
     (path "/e548561b-14bd-4e64-8562-e837f49c9f2f"
-      (reference "#PWR04") (unit 1) (value "POWER-GND") (footprint "")
+      (reference "#PWR0104") (unit 1) (value "POWER-GND") (footprint "")
     )
     (path "/c470ae0e-6742-4017-abb5-bba26fad9b9b"
-      (reference "#PWR05") (unit 1) (value "POWER-GND") (footprint "")
+      (reference "#PWR0105") (unit 1) (value "POWER-GND") (footprint "")
+    )
+    (path "/9ef92a8f-8f4c-46dd-be0c-47bafa44f512"
+      (reference "#PWR0106") (unit 1) (value "POWER-GND") (footprint "")
+    )
+    (path "/e9457c02-1887-4415-b9de-6d6efad5ec2d"
+      (reference "#PWR0107") (unit 1) (value "POWER-GND") (footprint "")
     )
     (path "/c7fd88e0-72a6-4454-ba59-3dff5184513c"
-      (reference "#PWR06") (unit 1) (value "POWER-GND") (footprint "")
+      (reference "#PWR0108") (unit 1) (value "POWER-GND") (footprint "")
     )
     (path "/fc54722e-43d3-4958-b314-96019cf0ccb6"
-      (reference "#PWR07") (unit 1) (value "POWER-VBAT") (footprint "")
-    )
-    (path "/e9457c02-1887-4415-b9de-6d6efad5ec2d"
-      (reference "#PWR0101") (unit 1) (value "POWER-GND") (footprint "")
+      (reference "#PWR0109") (unit 1) (value "POWER-VBAT") (footprint "")
     )
     (path "/1292386c-01d2-4aa5-a5bf-25821c6789db"
@@
     )
     (path "/32a690ff-98c8-4be1-b3d9-7e4cf3c6bc99"
-      (reference "K3") (unit 1) (value "I/O") (footprint "tronixio:HARWIN-M20-999034x")
+      (reference "K2") (unit 1) (value "I/O") (footprint "tronixio:HARWIN-M20-999034x")
     )
     (path "/5b4b00ae-6178-4d1f-920d-f4da9a4bc949"
-      (reference "K4") (unit 1) (value "I/O") (footprint "tronixio:HARWIN-M20-999064x")
+      (reference "K3") (unit 1) (value "I/O") (footprint "tronixio:HARWIN-M20-999064x")
+    )
+    (path "/d3cf96e2-b645-441e-b013-d9a2c067d09a"
+      (reference "TP1") (unit 1) (value "GND") (footprint "tronixio:KEYSTONE-2000-3")
     )
     (path "/967580e7-c183-44a2-9d11-d5df2d6657a8"

Commit message: Update
Parts:
- added C1: 10n, tronixio:CAPACITOR-SMD-1206, symbol tronixio:CAPACITOR-1206-10N
- added R1: 10K, tronixio:RESISTOR-SMD-1206, symbol tronixio:RESISTOR-1206-10K
- renumbered C1 to C2
Connections:
- net GND: now also C1.2
- net VCC: now also R1.1
- net at K1.6, U1.6 (~{E}): now also C1.1, R1.2
Other:
- moved on the sheet: C2, K3, U1
