File: Kicad/gpio-hc4053-header/hc4053-header.kicad_sch (KiCad schematic)
At the start: 9 parts, among them K1 GPIO IN, K2 I/O, K3 I/O, U1 74HC4053, U2 3M-SJ5376

Commit message: Up
Parts:
- C1: symbol tronixio:CAPACITOR-1206-10N -> tronixio:CAPACITOR-1206-100N-50V-5P-X7R; Mouser 80-C1206C103M5R -> 80-C1206C104J5R; Tolerance 20% -> 5%
- C2: symbol tronixio:CAPACITOR-1206-100N -> tronixio:CAPACITOR-1206-100N-50V-5P-X7R; Mouser 80-C1206C104M5R -> 80-C1206C104J5R; Tolerance 20% -> 5%
- R1: symbol tronixio:RESISTOR-1206-10K -> tronixio:RESISTOR-1206-10K-5P

Commit message: GPIO HC4053
Parts:
- C1: Name CAPACITOR-1206-10N -> (none)
- C2: Name CAPACITOR-1206-100N -> (none)
- K1: symbol tronixio:HARWIN-254-M-1X06-RIGHT-ANGLE -> tronixio:HARWIN-254-M-1X06-RIGHT-ANGLE-TH; Name HARWIN-254-M-1X06-RIGHT-ANGLE -> (none)
- K2: Name HARWIN-254-M-1X03-VERTICAL -> (none)
- K3: symbol tronixio:HARWIN-254-M-1X06-VERTICAL -> tronixio:HARWIN-254-M-1X06-VERTICAL-TH; Name HARWIN-254-M-1X06-VERTICAL -> (none)
- R1: value 10K -> 10k; Name RESISTOR-1206-10K -> (none)
- TP1: Name KEYSTONE-2000-3 -> (none)
- U1: symbol tronixio:74HC4053-SOIC-16 -> tronixio:NEXPERIA-74HC4053-SOIC16; Mouser 771-74HC4053D-T -> 771-74HC4053D; Name 74HC4053-SOIC-16 -> (none)
Connections:
- net POWER-GND renamed GND
- net POWER-VBAT renamed +VCC
Other:
- moved on the sheet: C1, C2, K1, K2, K3, R1, TP1, U1
