File: Kicad/gpio-mcp23008-led/mcp23008-led.kicad_sch (KiCad schematic)
At the start: 29 parts, among them K1 GPIO IN, K2 GPIO OUT, U1 MCP23008, U2 3M-SJ5376

Commit message: Up
Parts:
- C1: symbol tronixio:CAPACITOR-1206-100N -> tronixio:CAPACITOR-1206-100N-50V-5P-X7R; Mouser 80-C1206C104M5R -> 80-C1206C104J5R; Tolerance 20% -> 5%
- K2: symbol tronixio:SAMTEC-SSW-106-02-T-S-RA -> tronixio:SAMTEC-254-F-1X06-RIGHT-ANGLE; Mouser 200-SSW10602TSRA -> 200-SSW10603TSRA
- U1: I2C (none) -> @0x40
